Commit message: fix : added the new task, most of the logic done.
TODO: fix origin in the CADs, peg is not coming up as rigid_shape (is that an issue). Integrate the IK solving.

File: assets/industreal_kuka/urdf/kuka.urdf (robot description, URDF)
Before this commit: robot kuka_allegro, 10 links, 9 joints
Links:
- added link cross_peg, mass 1.41; collision mesh filename=../mesh/industreal_pegs/industreal_cross_peg.obj; visual mesh filename=../mesh/industreal_pegs/industreal_cross_peg.obj
Joints:
- added joint iiwa7_joint_peg: type fixed, parent iiwa7_link_ee, child cross_peg, origin xyz=0 0 0 rpy=0 0 0

Commit message: changes : commneted out peg link for now, brought the IK solver.
TODO: fix solver, fix indexing of rigid shape

File: assets/industreal_kuka/urdf/kuka.urdf (robot description, URDF)
Before this commit: robot kuka_allegro, 11 links, 10 joints
Links:
- link cross_peg: mass 1.41 -> None; geometry 
Joints:
- joint iiwa7_joint_peg: origin xyz=0 0 0 rpy=0 0 0 -> xyz=3.14 0 0 rpy=0 0 0

Commit message: change : goes to above pose and then goes to curriculum pose TODO: fix the transformation, some rotation error in the urdf

File: assets/industreal_kuka/urdf/kuka.urdf (robot description, URDF)
Before this commit: robot kuka_allegro, 11 links, 10 joints
Links:
- added link attachment; collision mesh filename=../mesh/industreal_pegs/industreal_cross_peg.obj; visual origin rpy=0 3.14 0 xyz=0 0 -0.03
Joints:
- added joint iiwa7_joint_attachment: type fixed, parent iiwa7_link_ee, child attachment, origin xyz=0 0 0 rpy=0 0 0
- joint iiwa7_joint_peg: origin xyz=3.14 0 0 rpy=0 0 0 -> xyz=0 0 -0.053 rpy=3.14 0 0
